File: rp2040-pico/rp2040-pico.kicad_sch (KiCad schematic)
At the start: 42 parts, among them J2 DIN41612_02x16_AB, J3 USB_C_Receptacle_USB2.0, J4 Micro_SD_Card_Det, Q7 DMG2305UX, Q8 DMG2305UX, U5 LM317_SOT-223

Commit message: Changed LM317 decoupling caps to non polarized
There is no need for C16, C17 or C18 to be polarized capacitors. As
such, they have been changed to be non polarized.

Signed-off-by: Matthew Nickson <mnickson@sidingsmedia.com>
Parts:
- C16, C17, C18: symbol Device:C_Polarized -> Device:C
Changed lines of the file:
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@@
     (pin "1")
   )
-  (symbol (lib_id "Device:C_Polarized") (at 71.12 153.67 0) (unit 1)
+  (symbol (lib_id "Device:C") (at 71.12 153.67 0) (unit 1)
     (in_bom yes) (on_board yes) (fields_autoplaced)
     (property "Reference" "C17" (id 0) (at 74.93 151.5109 0)
@@
     (pin "3")
   )
-  (symbol (lib_id "Device:C_Polarized") (at 29.21 148.59 0) (unit 1)
+  (symbol (lib_id "Device:C") (at 29.21 148.59 0) (unit 1)
     (in_bom yes) (on_board yes) (fields_autoplaced)
     (property "Reference" "C16" (id 0) (at 33.02 146.4309 0)
@@
     (pin "1")
   )
-  (symbol (lib_id "Device:C_Polarized") (at 86.36 148.59 0) (unit 1)
+  (symbol (lib_id "Device:C") (at 86.36 148.59 0) (unit 1)
     (in_bom yes) (on_board yes) (fields_autoplaced)
     (property "Reference" "C18" (id 0) (at 90.17 146.4309 0)

Commit message: Added device footprints
Signed-off-by: Matthew Nickson <mnickson@sidingsmedia.com>
Parts:
- C16, C17, C18: footprint (none) -> Capacitor_SMD:C_0402_1005Metric_Pad0.74x0.62mm_HandSolder
- D5, D6, D7: footprint (none) -> LED_SMD:LED_0603_1608Metric_Pad1.05x0.95mm_HandSolder
- J2: footprint (none) -> Connector_DIN:DIN41612_B2_2x16_Male_Horizontal_THT
- J3: footprint (none) -> Connector_USB:USB_C_Receptacle_Palconn_UTC16-G
- J4: footprint (none) -> Connector_Card:microSD_HC_Molex_104031-0811
- JP1: footprint (none) -> Jumper:SolderJumper-2_P1.3mm_Open_Pad1.0x1.5mm
- R24, R25, R26, R27, R28, R29: footprint (none) -> Resistor_SMD:R_0402_1005Metric_Pad0.72x0.64mm_HandSolder
- TP1, TP10, TP11, TP12, TP13, TP14, TP15, TP2, TP3, TP4, TP5, TP6, TP7, TP8, TP9: footprint (none) -> TestPoint:TestPoint_Pad_D1.0mm

Commit message: Updated schematic and started PCB development
Test points have been removed from the schematic where they were found
to be unnecessary or would make efficient placement of components
impossible. Most notable the test points connected to the flash chip.
These are not required as one can just probe the pins of the flash chip
with ease.

Some nets have also been labeled to assist in PCB development.

The componets have been roughly positioned on the PCB, grouped by their
function with the RP2040 related components being mostly connected.

Signed-off-by: Matthew Nickson <mnickson@sidingsmedia.com>
Parts:
- added SW3: SW_Push, Button_Switch_SMD:SW_SPST_B3U-1000P, symbol Switch:SW_Push
Connections:
- net GND: now also SW3.1
- net ~{RESET}: now also SW3.2
Changed lines of the file:
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@@
     (stroke (width 0) (type default) (color 0 0 0 0))
   )
-  (wire (pts (xy 115.57 66.04) (xy 128.27 66.04))
+  (wire (pts (xy 106.68 66.04) (xy 128.27 66.04))
     (stroke (width 0) (type default) (color 0 0 0 0))
   )
@@
     (stroke (width 0) (type default) (color 0 0 0 0))
   )
+  (wire (pts (xy 95.25 68.58) (xy 95.25 66.04))
+    (stroke (width 0) (type default) (color 0 0 0 0))
+  )
   (wire (pts (xy 71.12 137.16) (xy 86.36 137.16))
     (stroke (width 0) (type default) (color 0 0 0 0))
@@
   )
   (wire (pts (xy 92.71 123.19) (xy 107.95 123.19))
+    (stroke (width 0) (type default) (color 0 0 0 0))
+  )
+  (wire (pts (xy 95.25 66.04) (xy 96.52 66.04))
     (stroke (width 0) (type default) (color 0 0 0 0))
   )
@@
     (pin "2")
   )
+  (symbol (lib_id "Switch:SW_Push") (at 101.6 66.04 0) (unit 1)
+    (in_bom yes) (on_board yes) (fields_autoplaced)
+    (property "Reference" "SW3" (id 0) (at 101.6 58.42 0))
+    (property "Value" "SW_Push" (id 1) (at 101.6 60.96 0))
+    (property "Footprint" "Button_Switch_SMD:SW_SPST_B3U-1000P" (id 2) (at 101.6 60.96 0)
+      (effects (font (size 1.27 1.27)) hide)
+    )
+    (property "Datasheet" "~" (id 3) (at 101.6 60.96 0)
+      (effects (font (size 1.27 1.27)) hide)
+    )
+    (pin "1")
+    (pin "2")
+  )
   (symbol (lib_id "Connector:TestPoint") (at 200.66 27.94 0) (unit 1)
     (in_bom yes) (on_board yes)
@@
     (pin "1")
     (pin "2")
+  )
+  (symbol (lib_id "power:GND") (at 95.25 68.58 0) (unit 1)
+    (in_bom yes) (on_board yes) (fields_autoplaced)
+    (property "Reference" "#PWR016" (id 0) (at 95.25 74.93 0)
+      (effects (font (size 1.27 1.27)) hide)
+    )
+    (property "Value" "GND" (id 1) (at 95.25 73.66 0))
+    (property "Footprint" "" (id 2) (at 95.25 68.58 0)
+      (effects (font (size 1.27 1.27)) hide)
+    )
+    (property "Datasheet" "" (id 3) (at 95.25 68.58 0)
+      (effects (font (size 1.27 1.27)) hide)
+    )
+    (pin "1")
   )
   (symbol (lib_id "power:GND") (at 218.44 147.32 0) (unit 1)
@@
       (reference "#PWR015") (unit 1) (value "GND") (footprint "")
     )
-    (path "/db5cc6ec-32e5-4752-8117-f03b0aab0c5f/cee3619f-5813-4a8a-84c1-6c9d51fbd69c"
+    (path "/80aac459-56b6-4b66-8dec-d96ea435b309"
       (reference "#PWR016") (unit 1) (value "GND") (footprint "")
     )
@@
       (reference "D7") (unit 1) (value "LED") (footprint "LED_SMD:LED_0603_1608Metric_Pad1.05x0.95mm_HandSolder")
     )
-    (path "/db5cc6ec-32e5-4752-8117-f03b0aab0c5f/65348237-64b3-4600-9c46-1e9307c5b276"
-      (reference "J1") (unit 1) (value "Conn_01x03_Male") (footprint "Connector_PinHeader_2.54mm:PinHeader_1x03_P2.54mm_Vertical")
-    )
     (path "/96aba777-9ddb-4238-bfd5-baee0b5d77c4"
       (reference "J2") (unit 1) (value "DIN41612_02x16_AB") (footprint "Connector_DIN:DIN41612_B2_2x16_Male_Horizontal_THT")
@@
       (reference "SW2") (unit 1) (value "SW_Push") (footprint "Button_Switch_SMD:SW_SPST_B3U-1000P")
     )
+    (path "/1c586923-a4f8-419c-8159-e97918d9a438"
+      (reference "SW3") (unit 1) (value "SW_Push") (footprint "Button_Switch_SMD:SW_SPST_B3U-1000P")
+    )
     (path "/5a36cf36-9117-4f6d-92e6-f8f1c95ca265"
       (reference "TP1") (unit 1) (value "TestPoint") (footprint "TestPoint:TestPoint_Pad_D1.0mm")
@@
       (reference "TP17") (unit 1) (value "TestPoint") (footprint "TestPoint:TestPoint_Pad_D1.0mm")
     )
-    (path "/db5cc6ec-32e5-4752-8117-f03b0aab0c5f/4ff24516-46e4-4ee8-8082-06ceee2c4e3c"
-      (reference "TP18") (unit 1) (value "TestPoint") (footprint "TestPoint:TestPoint_Pad_D1.0mm")
-    )
-    (path "/db5cc6ec-32e5-4752-8117-f03b0aab0c5f/73df234c-5e93-438f-909a-0238f2798ac9"
-      (reference "TP19") (unit 1) (value "TestPoint") (footprint "TestPoint:TestPoint_Pad_D1.0mm")
-    )
-    (path "/db5cc6ec-32e5-4752-8117-f03b0aab0c5f/7ebdcac8-a73a-44ca-9f30-4517fac96b6f"
-      (reference "TP20") (unit 1) (value "TestPoint") (footprint "TestPoint:TestPoint_Pad_D1.0mm")
-    )
-    (path "/db5cc6ec-32e5-4752-8117-f03b0aab0c5f/9d6fd1fb-7a02-4cf1-b8f3-58d1a6a67d7c"
-      (reference "TP21") (unit 1) (value "TestPoint") (footprint "TestPoint:TestPoint_Pad_D1.0mm")
-    )
-    (path "/db5cc6ec-32e5-4752-8117-f03b0aab0c5f/a713af65-d5c4-4a46-89a2-9a2209456855"
-      (reference "TP22") (unit 1) (value "TestPoint") (footprint "TestPoint:TestPoint_Pad_D1.0mm")
-    )
-    (path "/db5cc6ec-32e5-4752-8117-f03b0aab0c5f/517e2ac2-9b40-465e-9216-1f3cb21a6077"
-      (reference "TP23") (unit 1) (value "TestPoint") (footprint "TestPoint:TestPoint_Pad_D1.0mm")
-    )
     (path "/db5cc6ec-32e5-4752-8117-f03b0aab0c5f/c086ba49-5b0b-443f-9ba0-e2ff7fc8b22f"
