File: rp2040-pico/mcu.kicad_sch (KiCad schematic)
At the start: 24 parts, among them J1 Conn_01x03_Male, Q6 DMG2305UX, U2 Pico, U3 RP2040, U4 W25Q128JVS, Y1 ABLS-12.000MHz-B4-T

Commit message: Added stat LEDs, BOOTSEL and reset button, SD card
3 LEDs have been added. One for indicating power and two for indicating
activity. Both activity LEDs are currently connected to the Pico/RP2040.
Buttons for boot selection and chip reset have been added to allow for
loading of firmware over USB. Support for a micro SD has also been
added. The card communicates with the Pico/RP2040 via the MCUs second
SPI interface and will store config files.

Signed-off-by: Matthew Nickson <mnickson@sidingsmedia.com>
Parts:
- added C19: C, symbol Device:C
- added R30, R31: 1K, symbol Device:R
- added SW2: SW_Push, symbol Switch:SW_Push
- added TP16, TP17, TP18, TP19, TP20, TP21, TP22, TP23, TP24: TestPoint, symbol Connector:TestPoint
Connections:
- net +3V3: now also R31.1
- net GND: now also C19.2, SW2.1
- net ~{RST}: now also C19.1, R31.2
- net ~{SD_DETECT}: now reaches U2.15 (GPIO11)
- net ~{SD_DETECT}: now also U3.14 (GPIO11)
- net SD_MISO: now reaches U2.16 (GPIO12)
- net SD_MISO: now also U3.15 (GPIO12)
- net ~{SD_CS}: now reaches U2.17 (GPIO13)
- net ~{SD_CS}: now also U3.16 (GPIO13)
- net SD_SCLK: now reaches U2.19 (GPIO14)
- net SD_SCLK: now also U3.17 (GPIO14)
- net SD_MOSI: now reaches U2.20 (GPIO15)
- net SD_MOSI: now also U3.18 (GPIO15)
- net LED1: now reaches U2.27 (GPIO21)
- net LED1: now also U3.32 (GPIO21)
- net LED2: now reaches U2.29 (GPIO22)
- net LED2: now also U3.34 (GPIO22)
- net at Q6.2 (S), U2.39 (VSYS): now also TP17.1
- net at Q6.1 (G), U2.40 (VBUS): now also TP16.1
- net at R20.2, U3.56 (QSPI_SS), U4.1 (~{CS}): now also R30.2, TP18.1
- net at U3.55 (QSPI_SD1), U4.2 (DO(IO1)): now also TP20.1
- net at U3.54 (QSPI_SD2), U4.3 (IO2): now also TP21.1
- net at U3.53 (QSPI_SD0), U4.5 (DI(IO0)): now also TP19.1
- net at U3.52 (QSPI_SCLK), U4.6 (CLK): now also TP23.1
- net at U3.51 (QSPI_SD3), U4.7 (IO3): now also TP22.1
- new net BOOTSEL: R30.1, SW2.2, TP24.1
- no-connect marks 4 -> 14
Other:
- note added: "Note: R20 is not required by this flash chip but may be required of a different flash is used."
- note added: "Place C15 close to pin 45"
- moved on the sheet: C13, R20, U4

Commit message: Assigned value to C19
Signed-off-by: Matthew Nickson <mnickson@sidingsmedia.com>
Parts:
- C19: value C -> 0.1u
Changed lines of the file:
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@@
       (effects (font (size 1.27 1.27)) (justify left))
     )
-    (property "Value" "C" (id 1) (at 149.86 186.6899 0)
+    (property "Value" "0.1u" (id 1) (at 149.86 186.6899 0)
       (effects (font (size 1.27 1.27)) (justify left))
     )

Commit message: Added device footprints
Signed-off-by: Matthew Nickson <mnickson@sidingsmedia.com>
Parts:
- C10, C11, C12, C13, C14, C15, C19, C2, C3, C4, C5, C6, C7, C8, C9: footprint (none) -> Capacitor_SMD:C_0402_1005Metric_Pad0.74x0.62mm_HandSolder
- J1: footprint (none) -> Connector_PinHeader_2.54mm:PinHeader_1x03_P2.54mm_Vertical
- R20, R21, R22, R23, R30, R31: footprint (none) -> Resistor_SMD:R_0402_1005Metric_Pad0.72x0.64mm_HandSolder
- SW2: footprint (none) -> Button_Switch_SMD:SW_SPST_B3U-1000P
- TP16, TP17, TP18, TP19, TP20, TP21, TP22, TP23, TP24: footprint (none) -> TestPoint:TestPoint_Pad_D1.0mm
- Y1: footprint (none) -> Crystal:Crystal_SMD_HC49-SD_HandSoldering
Changed lines of the file:
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@@
       (effects (font (size 1.27 1.27)) (justify left))
     )
-    (property "Footprint" "" (id 2) (at 242.2652 31.75 0)
+    (property "Footprint" "Capacitor_SMD:C_0402_1005Metric_Pad0.74x0.62mm_HandSolder" (id 2) (at 242.2652 31.75 0)
       (effects (font (size 1.27 1.27)) hide)
     )
@@
       (effects (font (size 1.27 1.27)) (justify left))
     )
-    (property "Footprint" "" (id 2) (at 207.9752 45.72 0)
+    (property "Footprint" "Capacitor_SMD:C_0402_1005Metric_Pad0.74x0.62mm_HandSolder" (id 2) (at 207.9752 45.72 0)
       (effects (font (size 1.27 1.27)) hide)
     )
@@
     (property "Reference" "R21" (id 0) (at 102.87 182.88 90))
     (property "Value" "1K" (id 1) (at 102.87 185.42 90))
-    (property "Footprint" "" (id 2) (at 102.87 191.008 90)
+    (property "Footprint" "Resistor_SMD:R_0402_1005Metric_Pad0.72x0.64mm_HandSolder" (id 2) (at 102.87 191.008 90)
       (effects (font (size 1.27 1.27)) hide)
     )
@@
       (effects (font (size 1.27 1.27)) (justify right))
     )
-    (property "Footprint" "" (id 2) (at 91.44 182.88 0)
+    (property "Footprint" "Crystal:Crystal_SMD_HC49-SD_HandSoldering" (id 2) (at 91.44 182.88 0)
       (effects (font (size 1.27 1.27)) hide)
     )
@@
       (effects (font (size 1.27 1.27)) (justify left))
     )
-    (property "Footprint" "" (id 2) (at 147.0152 189.23 0)
+    (property "Footprint" "Capacitor_SMD:C_0402_1005Metric_Pad0.74x0.62mm_HandSolder" (id 2) (at 147.0152 189.23 0)
       (effects (font (size 1.27 1.27)) hide)
     )
@@
     (property "Reference" "R22" (id 0) (at 226.06 53.34 90))
     (property "Value" "27R" (id 1) (at 226.06 55.88 90))
-    (property "Footprint" "" (id 2) (at 226.06 61.468 90)
+    (property "Footprint" "Resistor_SMD:R_0402_1005Metric_Pad0.72x0.64mm_HandSolder" (id 2) (at 226.06 61.468 90)
       (effects (font (size 1.27 1.27)) hide)
     )
@@
     (property "Reference" "C14" (id 0) (at 80.01 181.61 90))
     (property "Value" "27p" (id 1) (at 80.01 184.15 90))
-    (property "Footprint" "" (id 2) (at 83.82 188.2648 0)
+    (property "Footprint" "Capacitor_SMD:C_0402_1005Metric_Pad0.74x0.62mm_HandSolder" (id 2) (at 83.82 188.2648 0)
       (effects (font (size 1.27 1.27)) hide)
     )
@@
       (effects (font (size 1.27 1.27)) (justify left))
     )
-    (property "Footprint" "" (id 2) (at 253.6952 31.75 0)
+    (property "Footprint" "Capacitor_SMD:C_0402_1005Metric_Pad0.74x0.62mm_HandSolder" (id 2) (at 253.6952 31.75 0)
       (effects (font (size 1.27 1.27)) hide)
     )
@@
       (effects (font (size 1.27 1.27)) (justify left))
     )
-    (property "Footprint" "" (id 2) (at 139.3952 31.75 0)
+    (property "Footprint" "Capacitor_SMD:C_0402_1005Metric_Pad0.74x0.62mm_HandSolder" (id 2) (at 139.3952 31.75 0)
       (effects (font (size 1.27 1.27)) hide)
     )
@@
       (effects (font (size 1.27 1.27)) (justify left) hide)
     )
-    (property "Footprint" "" (id 2) (at 124.46 71.12 0)
+    (property "Footprint" "TestPoint:TestPoint_Pad_D1.0mm" (id 2) (at 124.46 71.12 0)
       (effects (font (size 1.27 1.27)) hide)
     )
@@
       (effects (font (size 1.27 1.27)) (justify left) hide)
     )
-    (property "Footprint" "" (id 2) (at 149.86 71.12 0)
+    (property "Footprint" "TestPoint:TestPoint_Pad_D1.0mm" (id 2) (at 149.86 71.12 0)
       (effects (font (size 1.27 1.27)) hide)
     )
@@
       (effects (font (size 1.27 1.27)) (justify left))
     )
-    (property "Footprint" "" (id 2) (at 176.2252 27.94 0)
+    (property "Footprint" "Capacitor_SMD:C_0402_1005Metric_Pad0.74x0.62mm_HandSolder" (id 2) (at 176.2252 27.94 0)
       (effects (font (size 1.27 1.27)) hide)
     )
@@
       (effects (font (size 1.27 1.27)) (justify left))
     )
-    (property "Footprint" "" (id 2) (at 98.7552 129.54 0)
+    (property "Footprint" "Capacitor_SMD:C_0402_1005Metric_Pad0.74x0.62mm_HandSolder" (id 2) (at 98.7552 129.54 0)
       (effects (font (size 1.27 1.27)) hide)
     )
@@
       (effects (font (size 1.27 1.27)) (justify left))
     )
-    (property "Footprint" "" (id 2) (at 230.8352 31.75 0)
+    (property "Footprint" "Capacitor_SMD:C_0402_1005Metric_Pad0.74x0.62mm_HandSolder" (id 2) (at 230.8352 31.75 0)
       (effects (font (size 1.27 1.27)) hide)
     )
@@
       (effects (font (size 1.27 1.27)) (justify right))
     )
-    (property "Footprint" "" (id 2) (at 38.1 185.42 0)
+    (property "Footprint" "Connector_PinHeader_2.54mm:PinHeader_1x03_P2.54mm_Vertical" (id 2) (at 38.1 185.42 0)
       (effects (font (size 1.27 1.27)) hide)
     )
@@
       (effects (font (size 1.27 1.27)) (justify left) hide)
     )
-    (property "Footprint" "" (id 2) (at 102.87 25.4 0)
+    (property "Footprint" "TestPoint:TestPoint_Pad_D1.0mm" (id 2) (at 102.87 25.4 0)
       (effects (font (size 1.27 1.27)) hide)
     )
@@
       (effects (font (size 1.27 1.27)) (justify left) hide)
     )
-    (property "Footprint" "" (id 2) (at 129.54 71.12 0)
+    (property "Footprint" "TestPoint:TestPoint_Pad_D1.0mm" (id 2) (at 129.54 71.12 0)
       (effects (font (size 1.27 1.27)) hide)
     )
@@
       (effects (font (size 1.27 1.27)) (justify left) hide)
     )
-    (property "Footprint" "" (id 2) (at 134.62 71.12 0)
+    (property "Footprint" "TestPoint:TestPoint_Pad_D1.0mm" (id 2) (at 134.62 71.12 0)
       (effects (font (size 1.27 1.27)) hide)
     )
@@
       (effects (font (size 1.27 1.27)) (justify left))
     )
-    (property "Footprint" "" (id 2) (at 219.4052 31.75 0)
+    (property "Footprint" "Capacitor_SMD:C_0402_1005Metric_Pad0.74x0.62mm_HandSolder" (id 2) (at 219.4052 31.75 0)
       (effects (font (size 1.27 1.27)) hide)
     )
@@
       (effects (font (size 1.27 1.27)) (justify left) hide)
     )
-    (property "Footprint" "" (id 2) (at 139.7 71.12 0)
+    (property "Footprint" "TestPoint:TestPoint_Pad_D1.0mm" (id 2) (at 139.7 71.12 0)
       (effects (font (size 1.27 1.27)) hide)
     )
@@
     (property "Reference" "R23" (id 0) (at 226.06 63.5 90))
     (property "Value" "27R" (id 1) (at 226.06 66.04 90))
-    (property "Footprint" "" (id 2) (at 226.06 71.628 90)
+    (property "Footprint" "Resistor_SMD:R_0402_1005Metric_Pad0.72x0.64mm_HandSolder" (id 2) (at 226.06 71.628 90)
       (effects (font (size 1.27 1.27)) hide)
     )
@@
       (effects (font (size 1.27 1.27)) (justify left) hide)
     )
-    (property "Footprint" "" (id 2) (at 144.78 71.12 0)
+    (property "Footprint" "TestPoint:TestPoint_Pad_D1.0mm" (id 2) (at 144.78 71.12 0)
       (effects (font (size 1.27 1.27)) hide)
     )
@@
       (effects (font (size 1.27 1.27)) (justify left))
     )
-    (property "Footprint" "" (id 2) (at 150.8252 31.75 0)
+    (property "Footprint" "Capacitor_SMD:C_0402_1005Metric_Pad0.74x0.62mm_HandSolder" (id 2) (at 150.8252 31.75 0)
       (effects (font (size 1.27 1.27)) hide)
     )
@@
     (property "Reference" "SW2" (id 0) (at 27.94 135.89 0))
     (property "Value" "SW_Push" (id 1) (at 27.94 138.43 0))
-    (property "Footprint" "" (id 2) (at 27.94 138.43 0)
+    (property "Footprint" "Button_Switch_SMD:SW_SPST_B3U-1000P" (id 2) (at 27.94 138.43 0)
       (effects (font (size 1.27 1.27)) hide)
     )
@@
     (property "Reference" "C4" (id 0) (at 80.01 168.91 90))
     (property "Value" "27p" (id 1) (at 80.01 171.45 90))
-    (property "Footprint" "" (id 2) (at 83.82 175.5648 0)
+    (property "Footprint" "Capacitor_SMD:C_0402_1005Metric_Pad0.74x0.62mm_HandSolder" (id 2) (at 83.82 175.5648 0)
       (effects (font (size 1.27 1.27)) hide)
     )
@@
       (effects (font (size 1.27 1.27)) (justify left) hide)
     )
-    (property "Footprint" "" (id 2) (at 39.37 146.05 0)
+    (property "Footprint" "TestPoint:TestPoint_Pad_D1.0mm" (id 2) (at 39.37 146.05 0)
       (effects (font (size 1.27 1.27)) hide)
     )
@@
       (effects (font (size 1.27 1.27)) (justify left))
     )
-    (property "Footprint" "" (id 2) (at 276.5552 31.75 0)
+    (property "Footprint" "Capacitor_SMD:C_0402_1005Metric_Pad0.74x0.62mm_HandSolder" (id 2) (at 276.5552 31.75 0)
       (effects (font (size 1.27 1.27)) hide)
     )
@@
       (effects (font (size 1.27 1.27)) (justify left))
     )
-    (property "Footprint" "" (id 2) (at 144.272 172.72 90)
+    (property "Footprint" "Resistor_SMD:R_0402_1005Metric_Pad0.72x0.64mm_HandSolder" (id 2) (at 144.272 172.72 90)
       (effects (font (size 1.27 1.27)) hide)
     )
@@
     (property "Reference" "R30" (id 0) (at 49.53 137.16 90))
     (property "Value" "1K" (id 1) (at 49.53 139.7 90))
-    (property "Footprint" "" (id 2) (at 49.53 145.288 90)
+    (property "Footprint" "Resistor_SMD:R_0402_1005Metric_Pad0.72x0.64mm_HandSolder" (id 2) (at 49.53 145.288 90)
       (effects (font (size 1.27 1.27)) hide)
     )
@@
       (effects (font (size 1.27 1.27)) (justify left))
     )
-    (property "Footprint" "" (id 2) (at 207.9752 31.75 0)
+    (property "Footprint" "Capacitor_SMD:C_0402_1005Metric_Pad0.74x0.62mm_HandSolder" (id 2) (at 207.9752 31.75 0)
       (effects (font (size 1.27 1.27)) hide)
     )
@@
       (effects (font (size 1.27 1.27)) (justify left) hide)
     )
-    (property "Footprint" "" (id 2) (at 92.71 38.1 0)
+    (property "Footprint" "TestPoint:TestPoint_Pad_D1.0mm" (id 2) (at 92.71 38.1 0)
       (effects (font (size 1.27 1.27)) hide)
     )
@@
       (effects (font (size 1.27 1.27)) (justify left))
     )
-    (property "Footprint" "" (id 2) (at 62.992 128.27 90)
+    (property "Footprint" "Resistor_SMD:R_0402_1005Metric_Pad0.72x0.64mm_HandSolder" (id 2) (at 62.992 128.27 90)
       (effects (font (size 1.27 1.27)) hide)
     )
@@
       (effects (font (size 1.27 1.27)) (justify left))
     )
-    (property "Footprint" "" (id 2) (at 265.1252 31.75 0)
-      (effects (font (size 1.27 1.27)) hide)
-    )
+    (property "Footprint" "Capacitor_SMD:C_0402_1005Metric_Pad0.74x0.62mm_HandSolder" (id 2) (at 265.1252 31.75 0)
+      (effects (font (size 1.27 1.27)) hide)
+    )

Commit message: Updated schematic and started PCB development
Test points have been removed from the schematic where they were found
to be unnecessary or would make efficient placement of components
impossible. Most notable the test points connected to the flash chip.
These are not required as one can just probe the pins of the flash chip
with ease.

Some nets have also been labeled to assist in PCB development.

The componets have been roughly positioned on the PCB, grouped by their
function with the RP2040 related components being mostly connected.

Signed-off-by: Matthew Nickson <mnickson@sidingsmedia.com>
Parts:
- removed J1: Conn_01x03_Male, Connector_PinHeader_2.54mm:PinHeader_1x03_P2.54mm_Vertical, symbol Connector:Conn_01x03_Male
- removed TP18, TP19, TP20, TP21, TP22, TP23: TestPoint, TestPoint:TestPoint_Pad_D1.0mm, symbol Connector:TestPoint
Connections:
- net CRYSTAL_OUT: now reaches R21.2, U3.21 (XOUT)
- net CRYSTAL_IN: now reaches C4.2, U3.20 (XIN), Y1.2
- net QSPI_SS: now reaches R20.2, R30.2, U3.56 (QSPI_SS), U4.1 (~{CS})
- net QSPI_SCLK: now reaches U3.52 (QSPI_SCLK), U4.6 (CLK)
- net QSPI_SD1: now reaches U3.55 (QSPI_SD1), U4.2 (DO(IO1))
- net QSPI_SD2: now reaches U3.54 (QSPI_SD2), U4.3 (IO2)
- net QSPI_SD0: now reaches U3.53 (QSPI_SD0), U4.5 (DI(IO0))
- net QSPI_SD3: now reaches U3.51 (QSPI_SD3), U4.7 (IO3)
Other:
- note added: "Note: There is no need for a seperate header to be included for the debug interface as one is included on the footprint of the pico."
- note removed: "Debug interface"
- moved on the sheet: R30, SW2, TP24
